Commit message: URDF completed. Cameras and LiDAR added

File: src/robot_ws_model_pkg/urdf/robot.urdf (robot description, URDF)
Before this commit: robot RAPID, 9 links, 8 joints
Links:
- added link front_camera_link; visual box size=0.010 0.03 0.03
- added link front_camera_link_optical
- added link laser; collision cylinder length=0.04 radius=0.05; visual cylinder length=0.04 radius=0.05
- added link rear_camera_link; visual box size=0.010 0.03 0.03
- added link rear_camera_link_optical
Joints:
- added joint front_camera_joint: type fixed, parent chassis_base, child front_camera_link, origin xyz=0.361 0.0866 0.06985 rpy=0 0 0
- added joint front_camera_optical_joint: type fixed, parent front_camera_link, child front_camera_link_optical, origin xyz=0 0 0 rpy=-1.5707963267948966 0 -1.5707963267948966
- added joint laser_joint: type fixed, parent lid, child laser, origin xyz=-0.09525 0 0.04 rpy=0 0 0
- added joint rear_camera_joint: type fixed, parent chassis_base, child rear_camera_link, origin xyz=-0.005 0.0866 0.06985 rpy=0 0 -3.14159265359
- added joint rear_camera_optical_joint: type fixed, parent rear_camera_link, child rear_camera_link_optical, origin xyz=0 0 0 rpy=-1.5707963267948966 0 -1.5707963267948966
